File: pcb/ai_pulsar.brd (EAGLE design)
At the start: 30.5 x 30.5 mm, 24 parts, among them IC1 DS1307SO8-TIGHT, IC3 74HCT245MTC, J2 1X05, U1 MIC5205-3.3

Commit message: routing finished
Parts:
- 3V-BATT: value (none) -> CR1220
- D1: value (none) -> PMEG2010AEB; device Ai_DiscreteSemis:SMA-403D -> Ai_DiscreteSemis:SOD-523
- XL1: value (none) -> CMR200T
- moved D1 22.7 mm to (6.32, 21.8), turned to 150 degrees
- moved C3 2.08 mm to (7.59, 15.2), turned to 180 degrees
- moved C1 1.90 mm to (7.59, 18.0), turned to 0 degrees
- moved U1 1.69 mm to (3.43, 21.8), turned to 150 degrees
- moved - 1.45 mm to (6.99, 25.4), turned to 40 degrees
- moved R5 0.51 mm to (27.2, 12.7)
- moved C4 0.25 mm to (7.59, 16.6), turned to 0 degrees
Routing:
- net N$5: track 0.00 -> 8.68 mm, vias 0 -> 2
- net 5V: track 56.6 -> 49.5 mm
- net 3V3: track 26.7 -> 31.2 mm
- net DTR: track 9.61 -> 13.2 mm
- net 3V3TXD: track 15.4 -> 18.4 mm
- net RESET: track 7.18 -> 8.20 mm
- net D: track 16.1 -> 17.0 mm
- net 3V3IO2: track 18.6 -> 19.3 mm
- net 5VIO2: track 10.4 -> 10.9 mm
- added copper zone on layer 1, net GND
- added copper zone on layer 16, net GND

Commit message: generated gerbers
Parts:
- moved U$6 33.0 mm to (13.8, 28.2), turned to 312 degrees
- moved U$9 26.9 mm to (20.0, 2.41), turned to 28 degrees
Routing:
- net 3V3IO5: track 20.9 -> 24.3 mm
- net N$4: track 15.9 -> 17.5 mm
- net RXI: track 10.7 -> 11.4 mm
Other:
- board text added: "+"
- board text added: "-"
- board text added: "CR1220 (RTC)"
- board text added: "D"
- board text added: "PULSAR"
- board text added: "Pasadena, CA"
- board text added: "www.acrobotic.com"
- board text removed: "0/TX"
- board text removed: "1/RX"
- board text removed: "2"
- board text removed: "3"
- board text removed: "3V3"
- board text removed: "4"
- board text removed: "5"
- board text removed: "6"
- board text removed: "DO"
- board text removed: "GND"
- board text removed: "Plug-n-Blink"
- board text removed: "RST"
- board text removed: "VIN"
- board text removed: "v1.2"
