File: pcb/ai_pulsar.sch (EAGLE design)
At the start: 25 parts, among them IC1 DS1307SO8-TIGHT, IC2 74HCT245MTC, J1 JST-3P-MALE, J2 1X05, U1 MIC5219-3.3

Commit message: updating
Parts:
- removed +, -, D: 1X01-PETAL, Ai_Connectors:1X01-PETAL
- removed D1: PMEG2010AEB, Ai_DiscreteSemis:DIODE-SCHOTTKYSMA-403D
- removed IC2: 74HCT245MTC, Ai_IC:74HCT245MTC
- added C10, C11, C12, C13, C14, C15, C16, C17, C18, C19, C20, C21, C22, C23, C24, C25, C26, C27, C28, C29, C6, C7, C8, C9: (no value), Ai_Passives:CAP0603
- added F1: (no value), Ai_Passives:PTCSMD
- added JS1: 1X02-SJ-NO, Ai_Connectors:1X02-SJ-NO
- added JS2: 1X02-SJ-NC, Ai_Connectors:1X02-SJ-NC
- added LED1, LED10, LED11, LED12, LED13, LED14, LED15, LED16, LED17, LED18, LED19, LED2, LED20, LED21, LED22, LED23, LED24, LED3, LED4, LED5, LED6, LED7, LED8, LED9: LED-WS2812B-SM, Ai_LED:LED-WS2812B-SM
- added LED25, LED26: (no value), Ai_LED:LED0603
- added Q1: BSS138, Ai_DiscreteSemis:FET-NMOS-BSS138
- added R10, R11: 330, Ai_Passives:RES0603
- added R6: 10K, Ai_Passives:RES0603
- added R7, R8, R9: 1K, Ai_Passives:RES0603
- added STANDOFF1, STANDOFF2, STANDOFF3, STANDOFF4: STAND-OFF4T, Ai_Electromechanical:STAND-OFF4T
- added U2: FT231X-Q, Ai_IC:FT231X-Q
- C1, C3: value 0.1uF -> 10uF
- C2: value 10uF -> 0.1uF
- C4: value 10uF -> (none)
- C5: value 100uF -> (none); device Ai_Passives:CAP-POLEIA3216 -> Ai_Passives:CAP0603
- J2: value 1X05 -> JST-2P-MALE; device Ai_Connectors:1X05 -> Ai_Connectors:JST-2P-MALE
- R1, R2: value 1K -> 22
- R5: value 1K -> 10K
Connections:
- removed net 3V3IO3: RFDUINO.P0.03/AIN4
- removed net 3V3IO4: RFDUINO.P0.04/AIN5
- removed net DTR: C1.2, J2.5
- removed net RESET: C1.1, RFDUINO.!RESET
- removed net RXI: J2.4, R1.2
- removed net TXO: J2.3, R2.2
- new net !RST: C5.1, RFDUINO.!RESET
- new net N$10: C5.2, U2.DTR#
- new net N$11: LED26.C, R11.2
- new net N$12: LED25.C, R10.2
- new net N$14: R10.1, U2.CBUS1
- new net N$15: R11.1, U2.CBUS2
- new net N$17: JS1.2
- new net N$2: R1.2, USB1.D-
- new net N$30: JS2.1, LED1.DI
- new net N$31: LED1.DO, LED2.DI
- new net N$6: R2.2, USB1.D+
- new net N$7: R9.1, U2.RXD
- new net N$8: R8.1, U2.TXD
- new net USBDM: R1.1, U2.USBDM
- new net USBDP: R2.1, U2.USBDP
- new net VCCIO: C4.2, LED25.A, LED26.A, U2.3V3OUT, U2.RESET#, U2.VCCIO
- net 3V3: now also C2.2, C3.1, Q1.G, R5.1; no longer C3.2, C4.1
- net 3V3IO2: now also Q1.S, R5.2; no longer IC2.A1
- net 3V3IO5: no longer RFDUINO.P0.05/AIN6
- net 3V3IO6: no longer RFDUINO.P0.06/AIN7
- net 3V3RXD: now also R9.2; no longer R1.1
- net 3V3TXD: now also R8.2; no longer R2.1
- net 5V: now also C1.1, C6.2, C7.2, F1.2, LED1.VDD, LED2.VDD, LED3.VDD, R6.1, U2.VCC; no longer +.1, C2.1, C5.A, D1.C, IC2.DIR, IC2.VCC, J2.2
- net 5VIO2: now also Q1.D, R6.2, R7.2; no longer IC2.B1, R5.2
- net D: now also JS1.1, JS2.2, R7.1; no longer D.1, R5.1
- net GND: now also C1.2, C2.1, C3.2, C4.1, C6.1, C7.1, LED1.VSS, LED2.VSS, U2.GND@13, U2.GND@21, U2.GND@3; no longer -.1, C2.2, C3.1, C4.2, C5.C, IC2.!OE, IC2.GND, J2.1
- net N$5: now also F1.1; no longer D1.A
Other:
- moved on the sheet: 3V-BATT, C1, C2, C3, C4, IC1, J1, R1, R2, R3, R4, R5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

Commit message: routing under way
Parts:
- added D1: DIODE-SCHOTTKY-DUAL, Ai_DiscreteSemis:DIODE-SCHOTTKY-DUAL
- added D2: (no value), Ai_DiscreteSemis:DIODE-SCHOTTKYSOD-523
- 3V-BATT: device Ai_Connectors:CR1220SMT -> Ai_Connectors:CR1025
Connections:
- new net +: D2.A, J2.+
- new net DI-1: LED6.DO, LED7.DI
- new net DI-2: LED18.DO, LED19.DI
- new net N$13: LED12.DO, LED13.DI
- new net N$16: LED2.DO, LED3.DI
- new net N$18: LED3.DO, LED4.DI
- new net N$19: LED4.DO, LED5.DI
- new net N$20: LED5.DO, LED6.DI
- new net N$21: LED7.DO, LED8.DI
- new net N$22: LED8.DO, LED9.DI
- new net N$23: LED10.DI, LED9.DO
- new net N$24: LED10.DO, LED11.DI
- new net N$25: LED11.DO, LED12.DI
- new net N$26: LED13.DO, LED14.DI
- new net N$27: LED14.DO, LED15.DI
- new net N$28: LED15.DO, LED16.DI
- new net N$29: LED16.DO, LED17.DI
- new net N$32: LED17.DO, LED18.DI
- new net N$33: LED19.DO, LED20.DI
- new net N$34: LED20.DO, LED21.DI
- new net N$35: LED21.DO, LED22.DI
- new net N$36: LED22.DO, LED23.DI
- new net N$37: LED23.DO, LED24.DI
- new net VBAT: D1.A2, D2.C
- new net VCC: C1.1, C10.2, C11.2, C12.2, C13.2, C14.2, C15.2, C16.2, C17.2, C18.2, C19.2, C20.2, C21.2, C22.2, C23.2, C24.2, C25.2, C26.2, C27.2, C28.2, C29.2, C6.2, C7.2, C8.2, C9.2, D1.CC, IC1.VCC, LED1.VDD, LED10.VDD, LED11.VDD, LED12.VDD, LED13.VDD, LED14.VDD, LED15.VDD, LED16.VDD, LED17.VDD, LED18.VDD, LED19.VDD, LED2.VDD, LED20.VDD, LED21.VDD, LED22.VDD, LED23.VDD, LED24.VDD, LED3.VDD, LED4.VDD, LED5.VDD, LED6.VDD, LED7.VDD, LED8.VDD, LED9.VDD, R6.1, U1.EN, U1.IN, U2.VCC
- net 5V: now also D1.A1; no longer C1.1, C6.2, C7.2, IC1.VCC, LED1.VDD, LED2.VDD, LED3.VDD, R6.1, U1.EN, U1.IN, U2.VCC
- net GND: now also C10.1, C11.1, C12.1, C13.1, C14.1, C15.1, C16.1, C17.1, C18.1, C19.1, C20.1, C21.1, C22.1, C23.1, C24.1, C25.1, C26.1, C27.1, C28.1, C29.1, C8.1, C9.1, J2.-, LED10.VSS, LED11.VSS, LED12.VSS, LED13.VSS, LED14.VSS, LED15.VSS, LED16.VSS, LED17.VSS, LED18.VSS, LED19.VSS, LED20.VSS, LED21.VSS, LED22.VSS, LED23.VSS, LED24.VSS, LED3.VSS, LED4.VSS, LED5.VSS, LED6.VSS, LED7.VSS, LED8.VSS, LED9.VSS
Other:
- moved on the sheet: 3V-BATT, C10, C11, C12, C13, C14, C15, C16, C17, C18, C19, C20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

Commit message: routed v1.3
Parts:
- removed U$6: AI-LOGOXS, Ai_Miscellany:AI-LOGOXS
- 3V-BATT: value CR1220 -> CR1025
- renumbered JS1 to STR, JS2 to RNG
Changed lines of the file:
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@@
 <part name="FRAME1" library="Ai_Miscellany" deviceset="FRAME-LETTER" device="">
 <attribute name="AUTHOR" value="A.I. HARDWARE SITH LORDS"/>
-<attribute name="REV" value="1.2"/>
+<attribute name="REV" value="1.3"/>
 </part>
 <part name="C1" library="Ai_Passives" deviceset="CAP" device="0603" value="10uF"/>
@@
 <part name="USB1" library="Ai_Connectors" deviceset="USB" device="MICROB-TH" value="USBMICROB-TH"/>
 <part name="GND7" library="Ai_Power" deviceset="GND" device=""/>
-<part name="U$6" library="Ai_Miscellany" deviceset="AI-LOGO" device="XS" value="AI-LOGOXS"/>
 <part name="RFDUINO" library="Ai_RF" deviceset="RFD22301" device=""/>
 <part name="GND1" library="Ai_Power" deviceset="GND" device=""/>
@@
 <part name="XL1" library="Ai_FrequencyControl" deviceset="CRYSTAL" device="CYL-2X6MM-SMT" value="CMR200T"/>
 <part name="U$3" library="Ai_Power" deviceset="3V3" device=""/>
-<part name="3V-BATT" library="Ai_Connectors" deviceset="CR1025" device="" value="CR1220"/>
+<part name="3V-BATT" library="Ai_Connectors" deviceset="CR1025" device="" value="CR1025"/>
 <part name="Q1" library="Ai_DiscreteSemis" deviceset="FET-NMOS" device="-BSS138" value="BSS138"/>
 <part name="U$5" library="Ai_Power" deviceset="3V3" device=""/>
@@
 <part name="STANDOFF3" library="Ai_Electromechanical" deviceset="STAND-OFF" device="4T"/>
 <part name="STANDOFF4" library="Ai_Electromechanical" deviceset="STAND-OFF" device="4T"/>
-<part name="JS1" library="Ai_Connectors" deviceset="1X02-SJ-NO" device=""/>
-<part name="JS2" library="Ai_Connectors" deviceset="1X02-SJ-NC" device=""/>
+<part name="STR" library="Ai_Connectors" deviceset="1X02-SJ-NO" device=""/>
+<part name="RNG" library="Ai_Connectors" deviceset="1X02-SJ-NC" device=""/>
 <part name="GND6" library="Ai_Power" deviceset="GND" device=""/>
 <part name="GND8" library="Ai_Power" deviceset="GND" device=""/>
@@
 <instance part="USB1" gate="G$1" x="8.89" y="106.68" rot="MR0"/>
 <instance part="GND7" gate="GND" x="68.58" y="83.82"/>
-<instance part="U$6" gate="G$1" x="1.27" y="1.27"/>
 <instance part="RFDUINO" gate="G$1" x="71.12" y="137.16"/>
 <instance part="GND1" gate="GND" x="17.78" y="97.79"/>
@@
 <instance part="STANDOFF3" gate="G$1" x="237.49" y="26.67"/>
 <instance part="STANDOFF4" gate="G$1" x="245.11" y="26.67"/>
-<instance part="JS1" gate="1" x="17.78" y="142.24" rot="R270"/>
-<instance part="JS2" gate="G$1" x="110.49" y="177.8" rot="R180"/>
+<instance part="STR" gate="1" x="17.78" y="142.24" rot="R270"/>
+<instance part="RNG" gate="G$1" x="110.49" y="177.8" rot="R180"/>
 <instance part="GND6" gate="GND" x="146.05" y="74.93"/>
 <instance part="GND8" gate="GND" x="167.64" y="49.53"/>
@@
 <label x="12.7" y="43.18" size="1.27" layer="95" font="vector" rot="R180" xref="yes"/>
 </segment>
+<segment>
+<wire x1="49.53" y1="137.16" x2="46.99" y2="137.16" width="0.1524" layer="91"/>
+<label x="46.99" y="137.16" size="1.27" layer="95" font="vector" ratio="10" rot="R180" xref="yes"/>
+</segment>
 </net>
 <net name="3V3IO6" class="0">
@@
 <label x="12.7" y="40.64" size="1.27" layer="95" font="vector" rot="R180" xref="yes"/>
 </segment>
+<segment>
+<wire x1="49.53" y1="134.62" x2="46.99" y2="134.62" width="0.1524" layer="91"/>
+<label x="46.99" y="134.62" size="1.27" layer="95" font="vector" ratio="10" rot="R180" xref="yes"/>
+</segment>
 </net>
 <net name="5VIO2" class="0">
@@
 <wire x1="19.05" y1="149.86" x2="17.78" y2="149.86" width="0.1524" layer="91"/>
 <label x="15.24" y="149.86" size="1.27" layer="95" font="vector" ratio="10" rot="R180" xref="yes"/>
-<pinref part="JS1" gate="1" pin="1"/>
+<pinref part="STR" gate="1" pin="1"/>
 <wire x1="17.78" y1="149.86" x2="15.24" y2="149.86" width="0.1524" layer="91"/>
 <wire x1="17.78" y1="147.32" x2="17.78" y2="149.86" width="0.1524" layer="91"/>
@@
 <segment>
 <label x="102.87" y="177.8" size="1.27" layer="95" font="vector" ratio="10" rot="R180" xref="yes"/>
-<pinref part="JS2" gate="G$1" pin="2"/>
+<pinref part="RNG" gate="G$1" pin="2"/>
 <wire x1="105.41" y1="177.8" x2="102.87" y2="177.8" width="0.1524" layer="91"/>
 </segment>
@@
 <net name="N$17" class="0">
 <segment>
-<pinref part="JS1" gate="1" pin="2"/>
+<pinref part="STR" gate="1" pin="2"/>
 <wire x1="17.78" y1="137.16" x2="17.78" y2="135.89" width="0.1524" layer="91"/>
 <wire x1="17.78" y1="135.89" x2="13.97" y2="135.89" width="0.1524" layer="91"/>
@@
 <segment>
 <pinref part="LED1" gate="G$1" pin="DI"/>
-<pinref part="JS2" gate="G$1" pin="1"/>
+<pinref part="RNG" gate="G$1" pin="1"/>
 <wire x1="115.57" y1="177.8" x2="116.84" y2="177.8" width="0.1524" layer="91"/>
 </segment>
@@
 </segment>
 </net>
+<net name="3V3IO3" class="0">
+<segment>
+<wire x1="49.53" y1="142.24" x2="46.99" y2="142.24" width="0.1524" layer="91"/>
+<label x="46.99" y="142.24" size="1.27" layer="95" font="vector" ratio="10" rot="R180" xref="yes"/>
+</segment>
+</net>
+<net name="3V3IO4" class="0">
+<segment>
+<wire x1="49.53" y1="139.7" x2="46.99" y2="139.7" width="0.1524" layer="91"/>
+<label x="46.99" y="139.7" size="1.27" layer="95" font="vector" ratio="10" rot="R180" xref="yes"/>
+</segment>
+</net>
