File: pcb/ai_pulsar.sch (EAGLE design)
At the start: 86 parts, among them IC1 DS1307SO8-TIGHT, J1 JST-3P-MALE, J2 JST-2P-MALE, Q1 BSS138, U1 MIC5219-3.3, U2 FT231X-Q

Commit message: fiddling with cutouts
Parts:
- removed D2: (no value), Ai_DiscreteSemis:DIODE-SCHOTTKYSOD-523
- removed Q1: BSS138, Ai_DiscreteSemis:FET-NMOS-BSS138
- removed R5, R6: 10K, Ai_Passives:RES0603
- R7: value 1K -> 330
- XL1: device Ai_FrequencyControl:CRYSTALCYL-2X6MM-SMT -> Ai_FrequencyControl:CRYSTALSMD
Connections:
- removed net +: D2.A, J2.+
- removed net 5VIO2: Q1.D, R6.2, R7.2
- new net 3V3IO3: RFDUINO.P0.03/AIN4
- new net 3V3IO4: RFDUINO.P0.04/AIN5
- net 3V3: no longer Q1.G, R5.1
- net 3V3IO2: now also R7.2; no longer Q1.S, R5.2
- net 3V3IO5: now also RFDUINO.P0.05/AIN6
- net 3V3IO6: now also RFDUINO.P0.06/AIN7
- net VBAT: now also J2.+; no longer D2.C
- net VCC: no longer R6.1
Other:
- moved on the sheet: R1, R2
Changed lines of the file:
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@@
 <part name="FRAME1" library="Ai_Miscellany" deviceset="FRAME-LETTER" device="">
 <attribute name="AUTHOR" value="A.I. HARDWARE SITH LORDS"/>
-<attribute name="REV" value="1.3"/>
+<attribute name="REV" value="1.4"/>
 </part>
 <part name="C1" library="Ai_Passives" deviceset="CAP" device="0603" value="10uF"/>
@@
 <part name="U1" library="Ai_Power" deviceset="MIC5219-*" device="" technology="3.3"/>
 <part name="GND2" library="Ai_Power" deviceset="GND" device=""/>
-<part name="R7" library="Ai_Passives" deviceset="RES" device="0603" value="1K"/>
+<part name="R7" library="Ai_Passives" deviceset="RES" device="0603" value="330"/>
 <part name="R4" library="Ai_Passives" deviceset="RES" device="0603" value="10K"/>
 <part name="R3" library="Ai_Passives" deviceset="RES" device="0603" value="10K"/>
-<part name="XL1" library="Ai_FrequencyControl" deviceset="CRYSTAL" device="CYL-2X6MM-SMT" value="CMR200T"/>
+<part name="XL1" library="Ai_FrequencyControl" deviceset="CRYSTAL" device="SMD" value="CMR200T"/>
 <part name="U$3" library="Ai_Power" deviceset="3V3" device=""/>
 <part name="3V-BATT" library="Ai_Connectors" deviceset="CR1025" device="" value="CR1025"/>
-<part name="Q1" library="Ai_DiscreteSemis" deviceset="FET-NMOS" device="-BSS138" value="BSS138"/>
-<part name="U$5" library="Ai_Power" deviceset="3V3" device=""/>
-<part name="R5" library="Ai_Passives" deviceset="RES" device="0603" value="10K"/>
-<part name="R6" library="Ai_Passives" deviceset="RES" device="0603" value="10K"/>
 <part name="LED1" library="Ai_LED" deviceset="LED-WS2812B" device="-SM"/>
 <part name="LED2" library="Ai_LED" deviceset="LED-WS2812B" device="-SM"/>
@@
 <part name="U$19" library="Ai_Power" deviceset="VBAT" device=""/>
 <part name="VCC1" library="Ai_Power" deviceset="VCC" device=""/>
-<part name="D2" library="Ai_DiscreteSemis" deviceset="DIODE-SCHOTTKY" device="SOD-523"/>
 <part name="VCC2" library="Ai_Power" deviceset="VCC" device=""/>
 <part name="VCC3" library="Ai_Power" deviceset="VCC" device=""/>
@@
 <part name="VCC6" library="Ai_Power" deviceset="VCC" device=""/>
 <part name="VCC7" library="Ai_Power" deviceset="VCC" device=""/>
-<part name="VCC8" library="Ai_Power" deviceset="VCC" device=""/>
 <part name="VCC9" library="Ai_Power" deviceset="VCC" device=""/>
 </parts>
@@
 <instance part="U$10" gate="G$1" x="13.97" y="140.97"/>
 <instance part="U$11" gate="G$1" x="30.48" y="113.03"/>
-<instance part="IC1" gate="G$1" x="33.02" y="45.72" rot="MR0"/>
+<instance part="IC1" gate="G$1" x="31.75" y="45.72" rot="MR0"/>
 <instance part="J1" gate="G$1" x="6.35" y="135.89" rot="MR270"/>
 <instance part="U1" gate="G$1" x="83.82" y="96.52"/>
@@
 <attribute name="VALUE" x="57.15" y="37.592" size="1.524" layer="96" font="vector" ratio="10" rot="MR0"/>
 </instance>
-<instance part="Q1" gate="G$1" x="22.86" y="158.75" rot="R270"/>
-<instance part="U$5" gate="G$1" x="15.24" y="175.26"/>
-<instance part="R5" gate="G$1" x="15.24" y="166.37" rot="R270"/>
-<instance part="R6" gate="G$1" x="29.21" y="166.37" rot="MR270"/>
 <instance part="LED1" gate="G$1" x="130.81" y="173.99" rot="MR0"/>
 <instance part="LED2" gate="G$1" x="130.81" y="156.21" rot="MR0"/>
@@
 <instance part="U2" gate="G$1" x="104.14" y="39.37"/>
 <instance part="J2" gate="G$1" x="10.16" y="85.09" rot="R90"/>
-<instance part="R1" gate="G$1" x="34.29" y="107.95" rot="MR0"/>
-<instance part="R2" gate="G$1" x="34.29" y="105.41" rot="MR0"/>
+<instance part="R1" gate="G$1" x="33.02" y="107.95" rot="MR0"/>
+<instance part="R2" gate="G$1" x="33.02" y="105.41" rot="MR0"/>
 <instance part="GND3" gate="GND" x="104.14" y="8.89"/>
 <instance part="C7" gate="G$1" x="170.18" y="59.69" rot="R180"/>
@@
 <instance part="GND12" gate="GND" x="212.09" y="74.93"/>
 <instance part="GND13" gate="GND" x="17.78" y="78.74"/>
-<instance part="U$17" gate="G$1" x="25.4" y="88.9"/>
+<instance part="U$17" gate="G$1" x="17.78" y="88.9"/>
 <instance part="D1" gate="G$1" x="43.18" y="82.55" rot="R270"/>
 <instance part="U$18" gate="G$1" x="43.18" y="88.9"/>
 <instance part="U$19" gate="G$1" x="36.83" y="88.9"/>
 <instance part="VCC1" gate="1" x="48.26" y="88.9"/>
-<instance part="D2" gate="G$1" x="20.32" y="86.36"/>
 <instance part="VCC2" gate="1" x="68.58" y="104.14"/>
 <instance part="VCC3" gate="1" x="20.32" y="60.96"/>
@@
 <instance part="VCC6" gate="1" x="147.32" y="180.34"/>
 <instance part="VCC7" gate="1" x="213.36" y="180.34"/>
-<instance part="VCC8" gate="1" x="29.21" y="175.26"/>
 <instance part="VCC9" gate="1" x="167.64" y="43.18"/>
 </instances>
@@
 <pinref part="U$3" gate="G$1" pin="3V3"/>
 </segment>
-<segment>
-<pinref part="U$5" gate="G$1" pin="3V3"/>
-<pinref part="R5" gate="G$1" pin="1"/>
-<wire x1="15.24" y1="171.45" x2="15.24" y2="172.72" width="0.1524" layer="91"/>
-<pinref part="Q1" gate="G$1" pin="G"/>
-<wire x1="15.24" y1="172.72" x2="15.24" y2="175.26" width="0.1524" layer="91"/>
-<wire x1="15.24" y1="172.72" x2="22.86" y2="172.72" width="0.1524" layer="91"/>
-<wire x1="22.86" y1="172.72" x2="22.86" y2="165.1" width="0.1524" layer="91"/>
-<junction x="15.24" y="172.72"/>
-</segment>
 </net>
 <net name="FACTORY" class="0">
@@
 </segment>
 <segment>
-<wire x1="15.24" y1="158.75" x2="12.7" y2="158.75" width="0.1524" layer="91"/>
-<label x="12.7" y="158.75" size="1.27" layer="95" font="vector" ratio="10" rot="R180" xref="yes"/>
-<pinref part="R5" gate="G$1" pin="2"/>
-<wire x1="15.24" y1="158.75" x2="15.24" y2="161.29" width="0.1524" layer="91"/>
-<pinref part="Q1" gate="G$1" pin="S"/>
-<wire x1="15.24" y1="158.75" x2="17.78" y2="158.75" width="0.1524" layer="91"/>
-<junction x="15.24" y="158.75"/>
+<wire x1="31.75" y1="149.86" x2="29.21" y2="149.86" width="0.1524" layer="91"/>
+<pinref part="R7" gate="G$1" pin="2"/>
+<label x="31.75" y="149.86" size="1.27" layer="95" font="vector" ratio="10" xref="yes"/>
 </segment>
 </net>
@@
 <wire x1="49.53" y1="137.16" x2="46.99" y2="137.16" width="0.1524" layer="91"/>
 <label x="46.99" y="137.16" size="1.27" layer="95" font="vector" ratio="10" rot="R180" xref="yes"/>
+<pinref part="RFDUINO" gate="G$1" pin="P0.05/AIN6"/>
 </segment>
 </net>
@@
 <wire x1="49.53" y1="134.62" x2="46.99" y2="134.62" width="0.1524" layer="91"/>
 <label x="46.99" y="134.62" size="1.27" layer="95" font="vector" ratio="10" rot="R180" xref="yes"/>
-</segment>
-</net>
-<net name="5VIO2" class="0">
-<segment>
-<label x="31.75" y="158.75" size="1.27" layer="95" font="vector" ratio="10" xref="yes"/>
-<pinref part="Q1" gate="G$1" pin="D"/>
-<pinref part="R6" gate="G$1" pin="2"/>
-<wire x1="27.94" y1="158.75" x2="29.21" y2="158.75" width="0.1524" layer="91"/>
-<wire x1="29.21" y1="158.75" x2="29.21" y2="161.29" width="0.1524" layer="91"/>
-<wire x1="29.21" y1="158.75" x2="31.75" y2="158.75" width="0.1524" layer="91"/>
-<junction x="29.21" y="158.75"/>
-</segment>
-<segment>
-<wire x1="31.75" y1="149.86" x2="29.21" y2="149.86" width="0.1524" layer="91"/>
-<pinref part="R7" gate="G$1" pin="2"/>
-<label x="31.75" y="149.86" size="1.27" layer="95" font="vector" xref="yes"/>
+<pinref part="RFDUINO" gate="G$1" pin="P0.06/AIN7"/>
 </segment>
 </net>
@@
 <segment>
 <label x="40.64" y="107.95" size="1.27" layer="95" font="vector" ratio="10" xref="yes"/>
-<wire x1="40.64" y1="107.95" x2="39.37" y2="107.95" width="0.1524" layer="91"/>
+<wire x1="40.64" y1="107.95" x2="38.1" y2="107.95" width="0.1524" layer="91"/>
 <pinref part="R1" gate="G$1" pin="1"/>
 </segment>
@@
 <pinref part="R2" gate="G$1" pin="1"/>
 <label x="40.64" y="105.41" size="1.27" layer="95" font="vector" ratio="10" xref="yes"/>
-<wire x1="39.37" y1="105.41" x2="40.64" y2="105.41" width="0.1524" layer="91"/>
+<wire x1="38.1" y1="105.41" x2="40.64" y2="105.41" width="0.1524" layer="91"/>
 </segment>
 <segment>
@@
 <pinref part="R1" gate="G$1" pin="2"/>
 <pinref part="USB1" gate="G$1" pin="D-"/>
-<wire x1="29.21" y1="107.95" x2="15.24" y2="107.95" width="0.1524" layer="91"/>
+<wire x1="27.94" y1="107.95" x2="15.24" y2="107.95" width="0.1524" layer="91"/>
 </segment>
 </net>
@@
 <segment>
 <pinref part="USB1" gate="G$1" pin="D+"/>
-<wire x1="15.24" y1="105.41" x2="29.21" y2="105.41" width="0.1524" layer="91"/>
+<wire x1="15.24" y1="105.41" x2="27.94" y2="105.41" width="0.1524" layer="91"/>
 <pinref part="R2" gate="G$1" pin="2"/>
 </segment>
@@
 <segment>
 <pinref part="U$17" gate="G$1" pin="VBAT"/>
-<wire x1="22.86" y1="86.36" x2="25.4" y2="86.36" width="0.1524" layer="91"/>
-<wire x1="25.4" y1="88.9" x2="25.4" y2="86.36" width="0.1524" layer="91"/>
-<pinref part="D2" gate="G$1" pin="C"/>
+<pinref part="J2" gate="G$1" pin="+"/>
+<wire x1="15.24" y1="86.36" x2="17.78" y2="86.36" width="0.1524" layer="91"/>
+<wire x1="17.78" y1="88.9" x2="17.78" y2="86.36" width="0.1524" layer="91"/>
 </segment>
 <segment>
@@
 </segment>
 <segment>
-<pinref part="R6" gate="G$1" pin="1"/>
-<wire x1="29.21" y1="171.45" x2="29.21" y2="175.26" width="0.1524" layer="91"/>
-<pinref part="VCC8" gate="1" pin="VCC"/>
-</segment>
-<segment>
 <wire x1="165.1" y1="40.64" x2="165.1" y2="41.91" width="0.1524" layer="91"/>
 <wire x1="165.1" y1="41.91" x2="167.64" y2="41.91" width="0.1524" layer="91"/>
@@
 </segment>
 </net>
-<net name="+" class="0">
-<segment>
-<pinref part="D2" gate="G$1" pin="A"/>
-<pinref part="J2" gate="G$1" pin="+"/>
-<wire x1="15.24" y1="86.36" x2="17.78" y2="86.36" width="0.1524" layer="91"/>
-</segment>
-</net>
 <net name="3V3IO3" class="0">
 <segment>
 <wire x1="49.53" y1="142.24" x2="46.99" y2="142.24" width="0.1524" layer="91"/>
 <label x="46.99" y="142.24" size="1.27" layer="95" font="vector" ratio="10" rot="R180" xref="yes"/>
+<pinref part="RFDUINO" gate="G$1" pin="P0.03/AIN4"/>
 </segment>
 </net>
@@
 <wire x1="49.53" y1="139.7" x2="46.99" y2="139.7" width="0.1524" layer="91"/>
 <label x="46.99" y="139.7" size="1.27" layer="95" font="vector" ratio="10" rot="R180" xref="yes"/>
-</segment>
-</net>
+<pinref part="RFDUINO" gate="G$1" pin="P0.04/AIN5"/>
+</segment>
+</net>

Commit message: bigger cutout for micro-B connector
Parts:
- C4, C5: value (none) -> 0.1uF
Changed lines of the file:
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@@
 <part name="LED23" library="Ai_LED" deviceset="LED-WS2812B" device="-SM"/>
 <part name="LED24" library="Ai_LED" deviceset="LED-WS2812B" device="-SM"/>
-<part name="C4" library="Ai_Passives" deviceset="CAP" device="0603"/>
+<part name="C4" library="Ai_Passives" deviceset="CAP" device="0603" value="0.1uF"/>
 <part name="R10" library="Ai_Passives" deviceset="RES" device="0603" value="330"/>
 <part name="U2" library="Ai_IC" deviceset="FT231X" device="-Q"/>
@@
 <part name="R9" library="Ai_Passives" deviceset="RES" device="0603" value="1K"/>
 <part name="R8" library="Ai_Passives" deviceset="RES" device="0603" value="1K"/>
-<part name="C5" library="Ai_Passives" deviceset="CAP" device="0603"/>
+<part name="C5" library="Ai_Passives" deviceset="CAP" device="0603" value="0.1uF"/>
 <part name="LED25" library="Ai_LED" deviceset="LED" device="0603"/>
 <part name="LED26" library="Ai_LED" deviceset="LED" device="0603"/>

Commit message: updating
Parts:
- removed R10, R11: 330, Ai_Passives:RES0603
- added R5: 100, Ai_Passives:RES0603
- added R6: 1K, Ai_Passives:RES0603
- D1: value DIODE-SCHOTTKY-DUAL -> PMEG4005CT
- R7: value 330 -> 1K
- R8, R9: value 1K -> 330
- XL1: value CMR200T -> MC146
Connections:
- net 3V3IO2: now also R5.2; no longer R7.2
- net 3V3RXD: now also R7.2; no longer R9.2
- net 3V3TXD: now also R6.2; no longer R8.2
- net D: now also R5.1; no longer R7.1
- net N$11: now also R9.2; no longer R11.2
- net N$12: now also R8.2; no longer R10.2
- net N$14: now also R8.1; no longer R10.1
- net N$15: now also R9.1; no longer R11.1
- net N$7: now also R7.1; no longer R9.1
- net N$8: now also R6.1; no longer R8.1
Other:
- moved on the sheet: R7, R8, R9
Changed lines of the file:
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@@
 <part name="FRAME1" library="Ai_Miscellany" deviceset="FRAME-LETTER" device="">
 <attribute name="AUTHOR" value="A.I. HARDWARE SITH LORDS"/>
-<attribute name="REV" value="1.4"/>
+<attribute name="REV" value="1.5"/>
 </part>
 <part name="C1" library="Ai_Passives" deviceset="CAP" device="0603" value="10uF"/>
@@
 <part name="U1" library="Ai_Power" deviceset="MIC5219-*" device="" technology="3.3"/>
 <part name="GND2" library="Ai_Power" deviceset="GND" device=""/>
-<part name="R7" library="Ai_Passives" deviceset="RES" device="0603" value="330"/>
+<part name="R5" library="Ai_Passives" deviceset="RES" device="0603" value="100"/>
 <part name="R4" library="Ai_Passives" deviceset="RES" device="0603" value="10K"/>
 <part name="R3" library="Ai_Passives" deviceset="RES" device="0603" value="10K"/>
-<part name="XL1" library="Ai_FrequencyControl" deviceset="CRYSTAL" device="SMD" value="CMR200T"/>
+<part name="XL1" library="Ai_FrequencyControl" deviceset="CRYSTAL" device="SMD" value="MC146"/>
 <part name="U$3" library="Ai_Power" deviceset="3V3" device=""/>
 <part name="3V-BATT" library="Ai_Connectors" deviceset="CR1025" device="" value="CR1025"/>
@@
 <part name="LED24" library="Ai_LED" deviceset="LED-WS2812B" device="-SM"/>
 <part name="C4" library="Ai_Passives" deviceset="CAP" device="0603" value="0.1uF"/>
-<part name="R10" library="Ai_Passives" deviceset="RES" device="0603" value="330"/>
+<part name="R8" library="Ai_Passives" deviceset="RES" device="0603" value="330"/>
 <part name="U2" library="Ai_IC" deviceset="FT231X" device="-Q"/>
 <part name="J2" library="Ai_Connectors" deviceset="JST-2P-MALE" device=""/>
@@
 <part name="GND3" library="Ai_Power" deviceset="GND" device=""/>
 <part name="C7" library="Ai_Passives" deviceset="CAP" device="0603"/>
-<part name="R9" library="Ai_Passives" deviceset="RES" device="0603" value="1K"/>
-<part name="R8" library="Ai_Passives" deviceset="RES" device="0603" value="1K"/>
+<part name="R7" library="Ai_Passives" deviceset="RES" device="0603" value="1K"/>
+<part name="R6" library="Ai_Passives" deviceset="RES" device="0603" value="1K"/>
 <part name="C5" library="Ai_Passives" deviceset="CAP" device="0603" value="0.1uF"/>
 <part name="LED25" library="Ai_LED" deviceset="LED" device="0603"/>
@@
 <part name="GND6" library="Ai_Power" deviceset="GND" device=""/>
 <part name="GND8" library="Ai_Power" deviceset="GND" device=""/>
-<part name="R11" library="Ai_Passives" deviceset="RES" device="0603" value="330"/>
+<part name="R9" library="Ai_Passives" deviceset="RES" device="0603" value="330"/>
 <part name="GND10" library="Ai_Power" deviceset="GND" device=""/>
 <part name="GND12" library="Ai_Power" deviceset="GND" device=""/>
 <part name="GND13" library="Ai_Power" deviceset="GND" device=""/>
 <part name="U$17" library="Ai_Power" deviceset="VBAT" device=""/>
-<part name="D1" library="Ai_DiscreteSemis" deviceset="DIODE-SCHOTTKY-DUAL" device=""/>
+<part name="D1" library="Ai_DiscreteSemis" deviceset="DIODE-SCHOTTKY-DUAL" device="" value="PMEG4005CT"/>
 <part name="U$18" library="Ai_Power" deviceset="5V" device=""/>
 <part name="U$19" library="Ai_Power" deviceset="VBAT" device=""/>
@@
 <instance part="U1" gate="G$1" x="83.82" y="96.52"/>
 <instance part="GND2" gate="GND" x="58.42" y="33.02"/>
-<instance part="R7" gate="G$1" x="24.13" y="149.86"/>
+<instance part="R5" gate="G$1" x="24.13" y="149.86"/>
 <instance part="R4" gate="G$1" x="17.78" y="53.34" rot="R270"/>
 <instance part="R3" gate="G$1" x="15.24" y="53.34" rot="R270"/>
@@
 <instance part="LED24" gate="G$1" x="228.6" y="173.99"/>
 <instance part="C4" gate="G$1" x="81.28" y="25.4" rot="R180"/>
-<instance part="R10" gate="G$1" x="127" y="35.56" rot="R90"/>
+<instance part="R8" gate="G$1" x="127" y="35.56" rot="R90"/>
 <instance part="U2" gate="G$1" x="104.14" y="39.37"/>
 <instance part="J2" gate="G$1" x="10.16" y="85.09" rot="R90"/>
@@
 <instance part="GND3" gate="GND" x="104.14" y="8.89"/>
 <instance part="C7" gate="G$1" x="170.18" y="59.69" rot="R180"/>
-<instance part="R9" gate="G$1" x="139.7" y="52.07"/>
-<instance part="R8" gate="G$1" x="139.7" y="54.61"/>
+<instance part="R7" gate="G$1" x="139.7" y="52.07"/>
+<instance part="R6" gate="G$1" x="139.7" y="54.61"/>
 <instance part="C5" gate="G$1" x="139.7" y="44.45" rot="R270"/>
 <instance part="LED25" gate="G$1" x="119.38" y="60.96" rot="R90"/>
@@
 <instance part="GND6" gate="GND" x="146.05" y="74.93"/>
 <instance part="GND8" gate="GND" x="167.64" y="49.53"/>
-<instance part="R11" gate="G$1" x="132.08" y="35.56" rot="R90"/>
+<instance part="R9" gate="G$1" x="132.08" y="35.56" rot="R90"/>
 <instance part="GND10" gate="GND" x="167.64" y="25.4"/>
 <instance part="GND12" gate="GND" x="212.09" y="74.93"/>
@@
 <wire x1="144.78" y1="54.61" x2="147.32" y2="54.61" width="0.1524" layer="91"/>
 <label x="147.32" y="54.61" size="1.27" layer="95" font="vector" ratio="10" xref="yes"/>
-<pinref part="R8" gate="G$1" pin="2"/>
+<pinref part="R6" gate="G$1" pin="2"/>
 </segment>
 </net>
@@
 <wire x1="144.78" y1="52.07" x2="147.32" y2="52.07" width="0.1524" layer="91"/>
 <label x="147.32" y="52.07" size="1.27" layer="95" font="vector" ratio="10" xref="yes"/>
-<pinref part="R9" gate="G$1" pin="2"/>
+<pinref part="R7" gate="G$1" pin="2"/>
 </segment>
 </net>
@@
 <segment>
 <wire x1="31.75" y1="149.86" x2="29.21" y2="149.86" width="0.1524" layer="91"/>
-<pinref part="R7" gate="G$1" pin="2"/>
+<pinref part="R5" gate="G$1" pin="2"/>
 <label x="31.75" y="149.86" size="1.27" layer="95" font="vector" ratio="10" xref="yes"/>
 </segment>
@@
 </segment>
 <segment>
-<pinref part="R7" gate="G$1" pin="1"/>
+<pinref part="R5" gate="G$1" pin="1"/>
 <wire x1="19.05" y1="149.86" x2="17.78" y2="149.86" width="0.1524" layer="91"/>
 <label x="15.24" y="149.86" size="1.27" layer="95" font="vector" ratio="10" rot="R180" xref="yes"/>
@@
 <segment>
 <pinref part="U2" gate="G$1" pin="RXD"/>
-<pinref part="R9" gate="G$1" pin="1"/>
+<pinref part="R7" gate="G$1" pin="1"/>
 <wire x1="134.62" y1="52.07" x2="124.46" y2="52.07" width="0.1524" layer="91"/>
 </segment>
@@
 <segment>
 <pinref part="U2" gate="G$1" pin="TXD"/>
-<pinref part="R8" gate="G$1" pin="1"/>
+<pinref part="R6" gate="G$1" pin="1"/>
 <wire x1="134.62" y1="54.61" x2="124.46" y2="54.61" width="0.1524" layer="91"/>
 </segment>
@@
 <net name="N$14" class="0">
 <segment>
-<pinref part="R10" gate="G$1" pin="1"/>
+<pinref part="R8" gate="G$1" pin="1"/>
 <pinref part="U2" gate="G$1" pin="CBUS1"/>
 <wire x1="124.46" y1="29.21" x2="127" y2="29.21" width="0.1524" layer="91"/>
@@
 <wire x1="124.46" y1="26.67" x2="132.08" y2="26.67" width="0.1524" layer="91"/>
 <wire x1="132.08" y1="26.67" x2="132.08" y2="30.48" width="0.1524" layer="91"/>
-<pinref part="R11" gate="G$1" pin="1"/>
+<pinref part="R9" gate="G$1" pin="1"/>
 </segment>
 </net>
@@
 <segment>
 <pinref part="LED26" gate="G$1" pin="C"/>
-<pinref part="R11" gate="G$1" pin="2"/>
+<pinref part="R9" gate="G$1" pin="2"/>
 <wire x1="130.81" y1="64.77" x2="132.08" y2="64.77" width="0.1524" layer="91"/>
 <wire x1="132.08" y1="64.77" x2="132.08" y2="40.64" width="0.1524" layer="91"/>
@@
 <segment>
 <pinref part="LED25" gate="G$1" pin="C"/>
-<pinref part="R10" gate="G$1" pin="2"/>
+<pinref part="R8" gate="G$1" pin="2"/>
 <wire x1="124.46" y1="60.96" x2="127" y2="60.96" width="0.1524" layer="91"/>
 <wire x1="127" y1="60.96" x2="127" y2="40.64" width="0.1524" layer="91"/>
